File: hardware/hardware_design/ESP32 IoT 4-layer PCB.kicad_pcb (KiCad board)
At the start: 4 copper layers, 83 parts, among them J1 SS-52400-003, J2 B2B-PH-SM4-TB, J3 GSD090012SEU, J4 Conn_01x04_Pin, J5 Conn_01x05_Pin, Q1 TEMT6000X01, Q2 BC817, Q3 BC817, U1 MCP73871-2CCI_ML, U2 MAX4466EXK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

Commit message: pcb layout completed
Parts:
- added C17: 10nF, Capacitor_SMD:C_0805_2012Metric, F.Cu at (180.7, 72.3)
- added C19: 1u, Capacitor_SMD:C_0805_2012Metric, F.Cu at (188.5, 69.8)
- C12, C3, C4, C7, C9: footprint Capacitor_Tantalum_SMD:CP_EIA-7132-20_AVX-U -> Capacitor_Tantalum_SMD:CP_EIA-3216-10_Kemet-I_HandSolder
- moved U3 135.7 mm to (243.4, 66.0)
- moved C22 134.4 mm to (224.3, 70.5)
- moved C21 132.9 mm to (226.2, 73.2), turned to 180 degrees
- moved S2 130.0 mm to (223.8, 67.2), turned to -90 degrees
- moved S1 125.0 mm to (225.9, 76.3), turned to 90 degrees
- moved R32 117.2 mm to (221.1, 67.2), turned to -90 degrees
- moved J3 117.2 mm to (238.6, 97.0)
- moved TP4 116.9 mm to (250.6, 81.6)
- moved J4 115.7 mm to (203.7, 59.6), turned to -90 degrees
- moved C12 108.6 mm to (234.6, 81.2), turned to 180 degrees
- moved C7 106.4 mm to (229.8, 64.8), turned to -90 degrees
- moved TP1 105.5 mm to (240.4, 78.1)
- moved C13 102.6 mm to (239.2, 81.2)
- moved R19 102.2 mm to (245.4, 80.7), turned to 90 degrees
- moved J5 100.7 mm to (179.1, 59.6), turned to 90 degrees
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Connections:
- C20 pad 1: GND -> Net-(U2-IN-)
- C4 pad 1: +3.3V -> Net-(U4-VBUS)
- MK1 pad OUT: Net-(U2-IN+) -> Net-(C17-Pad1)
- R28 pad 1: Net-(U2-IN+) -> Net-(C17-Pad1)
- R30 pad 1: GND -> Net-(C19-Pad1)
- R30 pad 2: GND -> Net-(U2-IN-)
- R31 pad 1: GND -> Net-(U2-IN-)
- U1 pad 1: (no net) -> +5V
- U1 pad 20: Net-(U1-OUT) -> +5V
- U2 pad 3: GND -> Net-(U2-IN-)
Routing:
- net /ESP32-C3 02/GPIO18: track 0.00 -> 73.9 mm, vias 0 -> 2
- net /ESP32-C3 02/GPIO19: track 0.00 -> 69.4 mm, vias 0 -> 2
- net /ESP32-C3 02/RX_TX: track 0.00 -> 66.2 mm, vias 0 -> 2
- net /ESP32-C3 02/GPIO8: track 0.00 -> 65.9 mm, vias 0 -> 2
- net /ESP32-C3 02/TX_RX: track 0.00 -> 65.3 mm, vias 0 -> 2
- net /ESP32-C3 02/SCL: track 0.00 -> 63.9 mm, vias 0 -> 2
- net /ESP32-C3 02/MISO_DO: track 0.00 -> 63.1 mm
- net /ESP32-C3 02/MOSI_DI: track 0.00 -> 63.0 mm
- net /ESP32-C3 02/SDA: track 0.00 -> 63.0 mm, vias 0 -> 2
- net +5V: track 0.00 -> 59.7 mm, vias 0 -> 6
- net +3.3V: track 0.00 -> 57.1 mm, vias 0 -> 39
- net /ESP32-C3 02/PHOTO_C: track 0.00 -> 54.5 mm, vias 0 -> 2
- net /ESP32-C3 02/BOOT: track 0.00 -> 53.7 mm, vias 0 -> 4
- net /ESP32-C3 02/MIC_OUT: track 0.00 -> 53.5 mm, vias 0 -> 2
- net /ESP32-C3 02/EN: track 0.00 -> 52.4 mm, vias 0 -> 2
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- added copper zone on F.Cu, net +3.3V
- added copper zone on In1.Cu, net +3.3V
- added copper zone on F.Cu, net +5V
- added copper zone on F.Cu, net /+5V_USB
- added copper zone on In1.Cu, net /+5V_USB
- added copper zone on F.Cu, net /VBAT
- added copper zone on F.Cu, net /VBUS
- added copper zone on In1.Cu, net /VBUS
- added copper zone on F.Cu, net GND
- added copper zone on In2.Cu, net GND
Other:
- board outline added: 86.2 x 55.3 mm
