File: hardware/hardware_design/ESP32 IoT 4-layer PCB.kicad_sch (KiCad schematic)
At the start: 25 parts, among them J1 SS-52400-003, J2 B2B-PH-SM4-TB, U1 MCP73871-2CCI_ML

Commit message: pcb layout completed
Parts:
- C3, C4: footprint Capacitor_Tantalum_SMD:CP_EIA-7132-20_AVX-U -> Capacitor_Tantalum_SMD:CP_EIA-3216-10_Kemet-I_HandSolder
Connections:
- net +5V: now also U1.20 (OUT)
Changed lines of the file:
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@@
 			)
 		)
-		(property "Footprint" "Capacitor_Tantalum_SMD:CP_EIA-7132-20_AVX-U"
+		(property "Footprint" "Capacitor_Tantalum_SMD:CP_EIA-3216-10_Kemet-I_HandSolder"
 			(at 108.1532 125.222 0)
 			(hide yes)
@@
 			)
 		)
-		(property "Footprint" "Capacitor_Tantalum_SMD:CP_EIA-7132-20_AVX-U"
+		(property "Footprint" "Capacitor_Tantalum_SMD:CP_EIA-3216-10_Kemet-I_HandSolder"
 			(at 47.9552 123.825 0)
 			(hide yes)
