File: hardware/hardware_design/esp32-c3 02.kicad_sch (KiCad schematic)
At the start: 30 parts, among them J3 GSD090012SEU, U3 ESP32-C3-WROOM-02-H4, U4 CP2102N-A02-GQFN20, U5 USBLC6-2SC6, U6 W25Q32JVSSIQ

Commit message: pcb layout completed
Parts:
- C12, C7, C9: footprint Capacitor_Tantalum_SMD:CP_EIA-7132-20_AVX-U -> Capacitor_Tantalum_SMD:CP_EIA-3216-10_Kemet-I_HandSolder
Changed lines of the file:
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@@
 			)
 		)
-		(property "Footprint" "Capacitor_Tantalum_SMD:CP_EIA-7132-20_AVX-U"
+		(property "Footprint" "Capacitor_Tantalum_SMD:CP_EIA-3216-10_Kemet-I_HandSolder"
 			(at 261.9248 138.43 0)
 			(hide yes)
@@
 			)
 		)
-		(property "Footprint" "Capacitor_Tantalum_SMD:CP_EIA-7132-20_AVX-U"
+		(property "Footprint" "Capacitor_Tantalum_SMD:CP_EIA-3216-10_Kemet-I_HandSolder"
 			(at 274.0152 64.77 0)
 			(hide yes)
@@
 			)
 		)
-		(property "Footprint" "Capacitor_Tantalum_SMD:CP_EIA-7132-20_AVX-U"
+		(property "Footprint" "Capacitor_Tantalum_SMD:CP_EIA-3216-10_Kemet-I_HandSolder"
 			(at 45.4152 78.105 0)
 			(hide yes)
